File: poor_man_DWM1001.brd (EAGLE design)
At the start: 32.6 x 26 mm, 18 parts, among them CN1 B2B-PH-K-S, IC1 E73_2G4M04S, U1 DWM1000_BREAKOUT, U3 MIC5205-3.3YM5-TR

Commit message: - Updated net names
Connections:
- net N$1 renamed GPIO_LED1_R
- net N$2 renamed GPIO_LED2_R
- net N$3 renamed GPIO_LED3_R
- net N$4 renamed GPIO_LED2
- net N$5 renamed GPIO_LED1
- net N$6 renamed GPIO_LED3
Changed lines of the file:
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@@
 <?xml version="1.0" encoding="utf-8"?>
 <!DOCTYPE eagle SYSTEM "eagle.dtd">
-<eagle version="8.6.0">
+<eagle version="9.0.0">
 <drawing>
 <settings>
@@
 <wire x1="8.349" y1="8.603" x2="7.493" y2="7.747" width="0.4064" layer="1"/>
 </signal>
-<signal name="N$1">
+<signal name="GPIO_LED1_R">
 <contactref element="R1" pad="2"/>
 <contactref element="LED1" pad="C"/>
@@
 <wire x1="2.159" y1="23.837" x2="2.198" y2="23.876" width="0.4064" layer="16"/>
 </signal>
-<signal name="N$2">
+<signal name="GPIO_LED2_R">
 <contactref element="R2" pad="2"/>
 <contactref element="LED2" pad="C"/>
@@
 <wire x1="3.175" y1="19.05" x2="2.782" y2="19.05" width="0.4064" layer="1"/>
 </signal>
-<signal name="N$3">
+<signal name="GPIO_LED3_R">
 <contactref element="R3" pad="2"/>
 <contactref element="LED3" pad="C"/>
@@
 <wire x1="2.782" y1="16.625" x2="2.198" y2="16.041" width="0.4064" layer="1"/>
 </signal>
-<signal name="N$4">
+<signal name="GPIO_LED2">
 <contactref element="R2" pad="1"/>
 <wire x1="8.922" y1="19.177" x2="7.779" y2="20.32" width="0.4064" layer="16"/>
@@
 <wire x1="22.606" y1="23.127" x2="22.847" y2="23.368" width="0.4064" layer="1"/>
 </signal>
-<signal name="N$5">
+<signal name="GPIO_LED1">
 <contactref element="R1" pad="1"/>
 <wire x1="21.463" y1="21.336" x2="20.701" y2="20.574" width="0.4064" layer="1"/>
@@
 <wire x1="21.535" y1="23.326" x2="21.463" y2="23.326" width="0.1524" layer="1"/>
 </signal>
-<signal name="N$6">
+<signal name="GPIO_LED3">
 <contactref element="R3" pad="1"/>
 <via x="3.81" y="13.335" extent="1-16" drill="0.5" diameter="1.05" shape="octagon"/>

Commit message: Added DWM1000 board
Parts:
- added C3: 100nF, rcl:C0603
- added C7, C8: 100pF, rcl:C0603
- added C9: 1uF, rcl:C0603
- added L1: 15nH, 3DR-GPS-LEA6-JST-v11-RELEASE:SPARKFUN_C0402
- added L2: 10uH, 3DR-GPS-LEA6-JST-v11-RELEASE:SPARKFUN_0603
- moved C1 0.38 mm to (25.3, 23.1)
- moved C2 0.38 mm to (23.1, 23.1)
- moved C4 0.38 mm to (14.2, 5.08)
- moved C5 0.38 mm to (20.6, 5.84)
- moved C6 0.38 mm to (17.0, 8.51)
- moved CN1 0.38 mm to (2.54, 2.16)
- moved IC1 0.38 mm to (10.0, 23.4)
- moved Q3 0.38 mm to (5.71, 1.91)
- moved R2 0.38 mm to (3.56, 19.7)
- moved R5 0.38 mm to (10.5, 1.27)
- moved SWD 0.38 mm to (2.86, 10.2)
- moved U1 0.38 mm to (5.38, 2.50)
- moved U3 0.38 mm to (17.1, 5.84)
- moved LED1 0.38 mm to (2.41, 20.8)
- moved LED2 0.38 mm to (2.41, 19.1)
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Connections:
- new net N$10: IC1.9
- new net N$11: IC1.10
- new net N$12: IC1.11
- new net N$13: L1.1, L2.2
- new net N$6: IC1.5
- new net N$7: IC1.6
- new net N$8: IC1.7
- new net N$9: IC1.8
- new net RESET: IC1.36
- net +3V3: now also U1.17
- net DCC: now also L2.1
- net DEC1: now also C3.1
- net DEC2: now also C7.1
- net DEC3: now also C8.1
- net DEC4: now also C9.1, L1.2
- net GND: now also C3.2, C7.2, C8.2, C9.2; no longer U1.17
Routing:
- net GND: track 90.8 -> 94.2 mm
